File: Hardware/Signal Generator/MainBoard.sch (EAGLE design)
At the start: 10 parts, among them U1 LMV358, U2 LMV358

Commit message: some ideas
Parts:
- added C3: 1.0uF, SparkFun-Capacitors:1.0UF-0402-16V-10%
- added IC1: AT89C52P6, atmel:AT89C52P6
- added Q1, Q2, Q3, Q4, Q5, Q6, Q7, Q8, Q9: (no value), semicon-smd-ipc:NPN-TRANSISTIOR-2COLSOT89
- added R10: 430k, SparkFun-Resistors:43KOHM-0603-1/10W-1%
- added R11: 4.3M, SparkFun-Resistors:43KOHM-0603-1/10W-1%
- added R12: 1M, pot:TRIM_1234-S64YW
- added R13, R15: 100K, SparkFun-Resistors:100KOHM-0402-1/16W-1%
- added R14, R16: 100k, pot:TRIM_1234-S64YW
- added R7: 430, SparkFun-Resistors:43KOHM-0603-1/10W-1%
- added R8: 43, SparkFun-Resistors:43KOHM-0603-1/10W-1%
- added R9: 43k, SparkFun-Resistors:43KOHM-0603-1/10W-1%
- added U3, U4: LMV358, SparkFun-IC-Amplifiers:LMV358SOIC
- R2: value 715 -> 10k
- R3: value 220k -> 100k
- R4: value 1M -> 100k
- R5: value 43k -> 4.3k
Connections:
- new net 100HZ: IC1G$1.P0.1AD1, Q5.B
- new net 100KHZ: IC1G$1.P0.4AD4, Q2.B
- new net 10HZ: IC1G$1.P0.0AD0, Q6.B
- new net 10KHZ: IC1G$1.P0.3AD3, Q3.B
- new net 1KHZ: IC1G$1.P0.2AD2, Q4.B
- new net 1MHZ: IC1G$1.P0.5AD5, Q1.B
- new net N$10: Q2.C, R7.1
- new net N$11: Q3.C, R5.1
- new net N$12: Q4.C, R9.1
- new net N$13: Q5.C, R10.1
- new net N$14: Q6.C, R11.1
- new net N$15: R14.E, R15.2, U4G2.-IN
- new net N$16: R16.E, U4G2.+IN
- new net N$21: IC1G$1.P1.2
- new net N$22: IC1G$1.P1.3
- new net N$23: IC1G$1.P1.4
- new net N$9: Q1.C, R8.1
- new net OUT: R14.S, U4G2.OUT
- new net SINE: C3.2, Q9.C, R13.2, U3G2.OUT
- new net SQUARE: Q7.C, R6.A, U1G2.OUT
- new net TRIANGLE: C2.2, Q8.C, R1.2, R12.E, U2G2.OUT
- net 0: now also R16.S, U3G2.+IN
- net N$2: now also Q1.E, Q2.E, Q3.E, Q4.E, Q5.E, Q6.E; no longer R5.1
- net N$3: now also R10.2, R11.2, R7.2, R8.2, R9.2
- net N$6: now also C3.1, R12.S, R13.1, U3G2.-IN; no longer R6.A, U1G2.OUT
- net N$8: now also Q7.E, Q8.E, Q9.E, R15.1; no longer C2.2, R1.2, U2G2.OUT
Other:
- note added: "DC offset"
- note added: "Digital Frequency range selector"
- note added: "amplifier +-15V"
- note removed: "R4 = R6"
- note removed: "Square Output"
- note removed: "Triangle Output"
- moved on the sheet: R5
